Commit message: init

File: zm_robot_description/urdf/zm_robot.urdf.xacro (robot description, xacro)
@@ -52,5 +52,4 @@
   <!-- Import Plugin -->
   <xacro:include filename="$(find zm_robot_description)/urdf/zm_robot_plugin.gazebo"/>
-  <!--xacro:include filename="$(find zm_robot_description)/urdf/zm_robot_plugin.gazebo"/-->
   <!-- Used for fixing robot to Gazebo 'base_link' -->
   <link name="base_footprint"/>
@@ -65,5 +64,5 @@
       <origin xyz="0 0 0" rpy="0 0 0"/>
       <geometry>
-        <mesh filename="package://zm_robot_description/meshes/agv_base.stl" scale="0.01 0.01 0.01"/>
+        <mesh filename="file://$(find zm_robot_description)/meshes/agv_base.stl" scale="0.01 0.01 0.01"/>
       </geometry>
     </collision>
@@ -71,5 +70,5 @@
       <origin xyz="0 0 0" rpy="0 0 0"/>
       <geometry>
-        <mesh filename="package://zm_robot_description/meshes/agv_base.stl" scale="0.01 0.01 0.01"/>
+        <mesh filename="file://$(find zm_robot_description)/meshes/agv_base.stl" scale="0.01 0.01 0.01"/>
       </geometry>
       <material name="orange"/>
@@ -93,5 +92,5 @@
       <origin xyz="0 0 0" rpy="0 0 0"/>
       <geometry>
-        <mesh filename="package://zm_robot_description/meshes/sick_s30b.stl" scale="0.01 0.01 0.01"/>
+        <mesh filename="file://$(find zm_robot_description)/meshes/sick_s30b.stl" scale="0.01 0.01 0.01"/>
       </geometry>
     </collision>
@@ -99,5 +98,5 @@
       <origin xyz="0 0 0" rpy="0 0 0"/>
       <geometry>
-        <mesh filename="package://zm_robot_description/meshes/sick_s30b.stl" scale="0.01 0.01 0.01"/>
+        <mesh filename="file://$(find zm_robot_description)/meshes/sick_s30b.stl" scale="0.01 0.01 0.01"/>
       </geometry>
       <material name="green"/>
@@ -121,5 +120,5 @@
       <origin xyz="0 0 0" rpy="0 0 0"/>
       <geometry>
-        <mesh filename="package://zm_robot_description/meshes/sick_s30b.stl" scale="0.01 0.01 0.01"/>
+        <mesh filename="file://$(find zm_robot_description)/meshes/sick_s30b.stl" scale="0.01 0.01 0.01"/>
       </geometry>
     </collision>
@@ -127,5 +126,5 @@
       <origin xyz="0 0 0" rpy="0 0 0"/>
       <geometry>
-        <mesh filename="package://zm_robot_description/meshes/sick_s30b.stl" scale="0.01 0.01 0.01"/>
+        <mesh filename="file://$(find zm_robot_description)/meshes/sick_s30b.stl" scale="0.01 0.01 0.01"/>
       </geometry>
       <material name="green"/>
@@ -150,5 +149,5 @@
       <origin xyz="0 0 0" rpy="0 0 0"/>
       <geometry>
-	      <mesh filename="package://zm_robot_description/meshes/kinect_v2.stl" scale="0.01 0.01 0.01"/>
+	      <mesh filename="file://$(find zm_robot_description)/meshes/kinect_v2.stl" scale="0.01 0.01 0.01"/>
       </geometry>
     </collision>
@@ -156,5 +155,5 @@
       <origin xyz="0 0 0" rpy="0 0 0"/>
       <geometry>
-	      <mesh filename="package://zm_robot_description/meshes/kinect_v2.stl" scale="0.01 0.01 0.01"/>
+	      <mesh filename="file://$(find zm_robot_description)/meshes/kinect_v2.stl" scale="0.01 0.01 0.01"/>
       </geometry>
       <material name="black"/>
@@ -179,5 +178,5 @@
       <origin xyz="0 0 0" rpy="0 0 0"/>
       <geometry>
-	      <mesh filename="package://zm_robot_description/meshes/IMU_sensor.stl" scale="0.01 0.01 0.01"/>
+	      <mesh filename="file://$(find zm_robot_description)/meshes/IMU_sensor.stl" scale="0.01 0.01 0.01"/>
       </geometry>
     </collision>
@@ -185,5 +184,5 @@
       <origin xyz="0 0 0" rpy="0 0 0"/>
       <geometry>
-	      <mesh filename="package://zm_robot_description/meshes/IMU_sensor.stl" scale="0.01 0.01 0.01"/>
+	      <mesh filename="file://$(find zm_robot_description)/meshes/IMU_sensor.stl" scale="0.01 0.01 0.01"/>
       </geometry>
       <material name="red"/>

File: zm_robot_description/urdf/zm_robot_roller.urdf.xacro (robot description, xacro)
@@ -14,5 +14,5 @@
 	  <visual>
 		<geometry>
-		  <mesh filename="package://zm_robot_description/meshes/mecanum_roller.stl" scale="0.01 0.01 0.01"/>
+		  <mesh filename="file://$(find zm_robot_description)/meshes/mecanum_roller.stl" scale="0.01 0.01 0.01"/>
 		</geometry>
 		<material name="black"/>
@@ -20,5 +20,5 @@
 	  <collision>
 		<geometry>
-		  <mesh filename="package://zm_robot_description/meshes/mecanum_roller.stl" scale="0.01 0.01 0.01"/>
+		  <mesh filename="file://$(find zm_robot_description)/meshes/mecanum_roller.stl" scale="0.01 0.01 0.01"/>
 		</geometry>
 	  </collision>

File: zm_robot_description/urdf/zm_robot_ultrasound.urdf.xacro (robot description, xacro)
@@ -13,5 +13,5 @@
 	  <visual>
 		<geometry>
-		  <mesh filename="package://zm_robot_description/meshes/ultrasound.stl" scale="0.1 0.1 0.1"/>
+		  <mesh filename="file://$(find zm_robot_description)/meshes/ultrasound.stl" scale="0.1 0.1 0.1"/>
 		</geometry>
 		<material name="blue"/>
@@ -19,5 +19,5 @@
 	  <collision>
 		<geometry>
-		  <mesh filename="package://zm_robot_description/meshes/ultrasound.stl" scale="0.1 0.1 0.1"/>
+		  <mesh filename="file://$(find zm_robot_description)/meshes/ultrasound.stl" scale="0.1 0.1 0.1"/>
 		</geometry>
 	  </collision>

File: zm_robot_description/urdf/zm_robot_wheel_LF.urdf.xacro (robot description, xacro)
@@ -13,5 +13,5 @@
 	  <visual>
 		<geometry>
-		  <mesh filename="package://zm_robot_description/meshes/mecanum_left_before.stl" scale="0.01 0.01 0.01"/>
+		  <mesh filename="file://$(find zm_robot_description)/meshes/mecanum_left_before.stl" scale="0.01 0.01 0.01"/>
 		</geometry>
 		<material name="white"/>
@@ -19,5 +19,5 @@
 	  <collision>
 		<geometry>
-		  <mesh filename="package://zm_robot_description/meshes/mecanum_left_before.stl" scale="0.01 0.01 0.01"/>
+		  <mesh filename="file://$(find zm_robot_description)/meshes/mecanum_left_before.stl" scale="0.01 0.01 0.01"/>
 		</geometry>
 	  </collision>
@@ -25,6 +25,6 @@
           <origin xyz="0.001 0 0" rpy="0 0 0"/>
           <mass value="1.7"/>
-          <inertia ixx="0.004248052" ixy="0.0" ixz="0.0"
-	               iyy="0.004248045" iyz="0.0" izz="0.004879970"/>
+          <inertia ixx="0.04248052" ixy="0.0" ixz="0.0"
+	               iyy="0.04248045" iyz="0.0" izz="0.04879970"/>
       </inertial>
 	</link>

File: zm_robot_description/urdf/zm_robot_wheel_LR.urdf.xacro (robot description, xacro)
@@ -13,5 +13,5 @@
 	  <visual>
 		<geometry>
-		  <mesh filename="package://zm_robot_description/meshes/mecanum_left_after.stl" scale="0.01 0.01 0.01"/>
+		  <mesh filename="file://$(find zm_robot_description)/meshes/mecanum_left_after.stl" scale="0.01 0.01 0.01"/>
 		</geometry>
 		<material name="white"/>
@@ -19,5 +19,5 @@
 	  <collision>
 		<geometry>
-		  <mesh filename="package://zm_robot_description/meshes/mecanum_left_after.stl" scale="0.01 0.01 0.01"/>
+		  <mesh filename="file://$(find zm_robot_description)/meshes/mecanum_left_after.stl" scale="0.01 0.01 0.01"/>
 		</geometry>
 	  </collision>
@@ -25,6 +25,6 @@
           <origin xyz="0.001 0 0" rpy="0 0 0"/>
           <mass value="1.7"/>
-          <inertia ixx="0.004248052" ixy="0.0" ixz="0.0"
-	               iyy="0.004248045" iyz="0.0" izz="0.004879970"/>
+          <inertia ixx="0.04248052" ixy="0.0" ixz="0.0"
+	               iyy="0.04248045" iyz="0.0" izz="0.04879970"/>
       </inertial>
 	</link>

File: zm_robot_description/urdf/zm_robot_wheel_RF.urdf.xacro (robot description, xacro)
@@ -13,5 +13,5 @@
 	  <visual>
 		<geometry>
-		  <mesh filename="package://zm_robot_description/meshes/mecanum_right_before.stl" scale="0.01 0.01 0.01"/>
+		  <mesh filename="file://$(find zm_robot_description)/meshes/mecanum_right_before.stl" scale="0.01 0.01 0.01"/>
 		</geometry>
 		<material name="white"/>
@@ -19,5 +19,5 @@
 	  <collision>
 		<geometry>
-		  <mesh filename="package://zm_robot_description/meshes/mecanum_right_before.stl" scale="0.01 0.01 0.01"/>
+		  <mesh filename="file://$(find zm_robot_description)/meshes/mecanum_right_before.stl" scale="0.01 0.01 0.01"/>
 		</geometry>
 	  </collision>
@@ -25,6 +25,6 @@
           <origin xyz="-0.001 0 0" rpy="0 0 0"/>
           <mass value="1.7"/>
-          <inertia ixx="0.004248052" ixy="0.0" ixz="0.0"
-	               iyy="0.004248045" iyz="0.0" izz="-0.004879970"/>
+          <inertia ixx="0.04248052" ixy="0.0" ixz="0.0"
+	               iyy="0.04248045" iyz="0.0" izz="-0.04879970"/>
       </inertial>
 	</link>

File: zm_robot_description/urdf/zm_robot_wheel_RR.urdf.xacro (robot description, xacro)
@@ -13,5 +13,5 @@
 	  <visual>
 		<geometry>
-		  <mesh filename="package://zm_robot_description/meshes/mecanum_right_after.stl" scale="0.01 0.01 0.01"/>
+		  <mesh filename="file://$(find zm_robot_description)/meshes/mecanum_right_after.stl" scale="0.01 0.01 0.01"/>
 		</geometry>
 		<material name="white"/>
@@ -19,5 +19,5 @@
 	  <collision>
 		<geometry>
-		  <mesh filename="package://zm_robot_description/meshes/mecanum_right_after.stl" scale="0.01 0.01 0.01"/>
+		  <mesh filename="file://$(find zm_robot_description)/meshes/mecanum_right_after.stl" scale="0.01 0.01 0.01"/>
 		</geometry>
 	  </collision>
@@ -25,6 +25,6 @@
           <origin xyz="-0.001 0 0" rpy="0 0 0"/>
           <mass value="1.7"/>
-          <inertia ixx="0.004248052" ixy="0.0" ixz="0.0"
-	               iyy="0.004248045" iyz="0.0" izz="-0.004879970"/>
+          <inertia ixx="0.04248052" ixy="0.0" ixz="0.0"
+	               iyy="0.04248045" iyz="0.0" izz="-0.04879970"/>
       </inertial>
 	</link>
